Commit message: chassis is fully defined

File: robot_nav_ai/robot/robot.urdf (robot description, URDF)
Before this commit: robot nav_robot, 8 links, 7 joints
Links:
- added link base_footprint
- link base_link: geometry collision box size=0.40 0.30 0.10; visual box size=0.02 0.30 0.06
Joints:
- added joint base_footprint_joint: type fixed, parent base_footprint, child base_link, origin xyz=0 0 0.05 rpy=0 0 0

Commit message: wheel sections with corrected inertia, multi-layer visuals, contact properties, and joint limits

File: robot_nav_ai/robot/robot.urdf (robot description, URDF)
Before this commit: robot nav_robot, 9 links, 8 joints
Links:
- link left_wheel: geometry collision cylinder length=0.04 radius=0.05; visual box size=0.008 0.003 0.040
- link right_wheel: geometry collision cylinder length=0.04 radius=0.05; visual box size=0.008 0.003 0.040
Joints:
- joint left_wheel_joint: limit (none) -> effort=10.0 velocity=10.0; origin xyz=0.1 0.17 0.0 rpy=0 0 0 -> xyz=0.0 0.17 0.0 rpy=0 0 0
- joint right_wheel_joint: limit (none) -> effort=10.0 velocity=10.0; origin xyz=0.1 -0.17 0.0 rpy=0 0 0 -> xyz=0.0 -0.17 0.0 rpy=0 0 0

Commit message: lidar setup

File: robot_nav_ai/robot/robot.urdf (robot description, URDF)
Before this commit: robot nav_robot, 9 links, 8 joints
Links:
- removed link caster_wheel
- added link caster_ball, mass 0.08; collision sphere radius=0.03; visual cylinder length=0.006 radius=0.031
- added link caster_stem, mass 0.05; visual box size=0.012 0.040 0.008; visual cylinder length=0.02 radius=0.006
- added link lidar_mount, mass 0.15; collision box size=0.06 0.06 0.02; visual box size=0.06 0.06 0.02
- link lidar_link: geometry collision cylinder length=0.040 radius=0.042; visual cylinder length=0.004 radius=0.020
Joints:
- removed joint caster_joint
- added joint caster_ball_joint: type fixed, parent caster_stem, child caster_ball, origin xyz=0 0.0 -0.03 rpy=0 0 0
- added joint caster_stem_joint: type fixed, parent base_link, child caster_stem, origin xyz=0.15 0.0 -0.05 rpy=0 0 0
- added joint lidar_mount_joint: type fixed, parent base_link, child lidar_mount, origin xyz=0.10 0.0 0.06 rpy=0 0 0
- joint lidar_joint: origin xyz=0.05 0.0 0.12 rpy=0 0 0 -> xyz=0 0 0.03 rpy=0 0 0; parent base_link -> lidar_mount
